File: board/wallet.kicad_pcb (KiCad board)
At the start: 4 copper layers, 48 x 85 mm, 136 parts, among them J1 TYPE-C-31-M-12, U1 BQ25185DLHR, U10 SN74LVC1T45DBVR, U11 E73-2G4M08S1C, U12 ME6211C28M5G-N, U13 TPS60230RGTR, U14 TLV75801PDBVR, U15 MAX17048G+T10, U2 TPS63802DLAR, U3 XC6206P332MR-G, U4 STM32U585VIT6Q, U5 SE050E2HQ1/Z01Z3Z, U6 TS3USB221ARSER, U7 SN74LVC1G02DBVR(UMW), U8 TPS22917DBVR, U9 SN74LVC1T45DBVR, Y1 Q13FC13500049

Commit message: Ratsnest-optimized placement: autorouter completes every net
- newBoard.py runs optimizePlacement.py after legalization (radius 7 mm):
  crossings 460 -> 286, airwire 1871 -> 1714 mm
- scripts/trialRoute.sh: autoroutes a copy with KiCadRoutingTools and reports
  failed nets / vias. Seed 3 failed / 209 vias; this board 0 failed / 207.
  Radius 4 and MCU pin swaps were measured worse and are not applied.
- RADIO light under the south-west hole, out of the west bridge into the chin;
  hole rings 2.6 mm (M2 head); a reserved slot keeps the SECURE ELEMENT label
- UV art rebuilt for this placement

Co-Authored-By: Claude Opus 5.5 <noreply@anthropic.com>
Parts:
- moved R_RLED 11.1 mm to (5.10, 64.7), turned to 0 degrees
- moved D_RADIO 8.14 mm to (5.34, 62.9), turned to 0 degrees
- moved U15 6.96 mm to (43.3, 49.9), turned to 0 degrees
- moved R_SESDA 6.95 mm to (11.8, 29.1), turned to -90 degrees
- moved U6 6.80 mm to (23.5, 65.6), turned to -90 degrees
- moved Q_BTN 6.80 mm to (40.3, 43.9), turned to 180 degrees
- moved R_BTNN 6.80 mm to (40.3, 47.4), turned to -90 degrees
- moved R_CE 6.73 mm to (31.9, 60.8), turned to 180 degrees
- moved C_RTC 6.71 mm to (34.2, 75.0), turned to 0 degrees
- moved C_U9B 6.58 mm to (2.20, 32.5), turned to 0 degrees
- moved R_ILIM 6.58 mm to (29.3, 64.8), turned to 180 degrees
- moved C_EN 6.52 mm to (45.3, 31.0), turned to 0 degrees
- moved R_TS 6.52 mm to (32.4, 65.3)
- moved C_U10B 6.50 mm to (3.50, 26.0), turned to 0 degrees
- moved R_CSCL 6.50 mm to (32.8, 12.1), turned to 0 degrees
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