File: board/wallet.kicad_pcb (KiCad board)
At the start: 4 copper layers, 48 x 85 mm, 108 parts, among them J1 TYPE-C-31-M-12, U1 BQ25185DLHR, U11 E73-2G4M08S1C, U12 ME6211C28M5G-N, U13 TPS60230RGTR, U14 TLV70313DBVR, U15 MAX17048G+T10, U2 TPS63802DLAR, U4 STM32U585VIT6Q, U5 SE050E2HQ1/Z01Z3Z, U6 TS3USB221ARSER, U7 SN74LVC1G02DBVR(UMW), U8 TPS22917DBVR, U9 TXU0202DCUR

Commit message: Owner: SE rotated toward the MCU, pull-ups inline, SE block and charger TS routed
Secure element turned -90 deg so SDA/SCL/ENA face the MCU's west pins; its
three pull-ups in a column between the two, both caps moved; SE wiring, CHG_TS
and BAT routed by hand; R_TS beside the charger. Three GND fanout vias next to
GND pads removed (the pour plus stitching does that job).

Co-Authored-By: Claude Opus 5.5 <noreply@anthropic.com>
Parts:
- moved R_TS 10.2 mm to (36.3, 74.8)
- moved C_SEVCC 5.53 mm to (4.34, 29.8), turned to -90 degrees
- moved R_SEENA 4.34 mm to (10.9, 31.5), turned to 0 degrees
- moved R_SESDA 3.82 mm to (10.8, 29.3), turned to 0 degrees
- moved R_SESCL 3.70 mm to (10.8, 30.3), turned to 0 degrees
- moved C_SEIN 2.64 mm to (8.09, 31.9), turned to 0 degrees
- moved U5 1.58 mm to (7.64, 29.1), turned to -90 degrees
Routing:
- net V3V3: track 87.9 -> 112.7 mm
- net SE_SCL: track 1.34 -> 7.46 mm
- net SE_ENA: track 2.35 -> 7.58 mm
- net SE_SDA: track 1.23 -> 6.43 mm
- net GND: track 85.7 -> 81.9 mm, vias 70 -> 67
- net CHG_TS: track 0.00 -> 1.26 mm
