File: board/wallet.kicad_pcb (KiCad board)
At the start: 4 copper layers, 48 x 85 mm, 108 parts, among them J1 TYPE-C-31-M-12, U1 BQ25185DLHR, U11 E73-2G4M08S1C, U12 ME6211C28M5G-N, U13 TPS60230RGTR, U14 TLV70313DBVR, U15 MAX17048G+T10, U2 TPS63802DLAR, U4 STM32U585VIT6Q, U5 SE050E2HQ1/Z01Z3Z, U6 TS3USB221ARSER, U7 SN74LVC1G02DBVR(UMW), U8 TPS22917DBVR, U9 TXU0202DCUR

Commit message: Second secure element from a second vendor: Infineon OPTIGA Trust M V3
Key model: two non-extractable keys, one in the NXP SE050 and an independent
P-256 key in the OPTIGA (CC EAL6+ hardware), so one vendor's silicon break
yields one key, not the device's signing authority; the account treats the
device as one owner needing both (research.md).

Hardware: SLS32AIA010MK (C1518668, 0 at JLC; V1 SLS32AIA010MH C539250 on the
same land has 60) on the secure elements' own I2C4 bus at 0x30 beside the
SE050's 0x48, RST from PD14 (pulled high, 100k), 100 nF at VCC; pins from the
data sheet Rev 3.10 Table 6, the centre pad (not in the table) soldered but
unconnected. KiCad's DFN-10 3x3 EP1.7x2.5 land matches Infineon's outline and
JLC's land. Placed north of the SE050 by place_block; all four rotations
routed to 42-50 mm with 4-5 vias (the part puts SDA on the opposite row from
SCL/RST), 270 deg kept.

Stitching regenerated around the new part (humanRouter GND pass), no GND
pad-to-via ties beyond the 9 kept ones; router's stray V3V3 vias removed.

Tools: syncBoard adds parts on the back with the board's text style
(newBoard.style_text); checkParts compares copper pads only, so a land's
paste-only apertures no longer read as extra pads (the U13/U15 waivers that
existed only for that are gone).

Unconnected 5 (USB MCU pair, RADIO_TXD, AIRGAP x2); 0 copper DRC; nets, AF,
sync, pin tables (17 parts), FPC, lands pass.

Co-Authored-By: Claude Opus 5.5 <noreply@anthropic.com>
Parts:
- added C_OPT: 100nF, Capacitor_SMD:C_0402_1005Metric, B.Cu at (2.46, 26.1)
- added R_OPTRST: 100k, Resistor_SMD:R_0402_1005Metric, B.Cu at (7.71, 25.1)
- added U16: SLS32AIA010MK, Package_DFN_QFN:DFN-10-1EP_3x3mm_P0.5mm_EP1.7x2.5mm, B.Cu at (5.25, 24.5)
Connections:
- U4 pad 61: (no net) -> OPTIGA_RST
Routing:
- net GND: track 52.7 -> 87.1 mm, vias 251 -> 242
- net OPTIGA_RST: track 0.00 -> 12.5 mm
- net SE_SDA: track 6.43 -> 16.2 mm, vias 0 -> 2
- net SE_SCL: track 7.46 -> 13.8 mm, vias 0 -> 2
- net V3V3: track 135.2 -> 138.0 mm, vias 42 -> 45
