File: board/wallet.kicad_pcb (KiCad board)
At the start: 4 copper layers, 48 x 85 mm, 111 parts, among them J1 TYPE-C-31-M-12, U1 BQ25185DLHR, U11 E73-2G4M08S1C, U12 ME6211C28M5G-N, U13 TPS60230RGTR, U14 TLV70313DBVR, U15 MAX17048G+T10, U16 SLS32AIA010MK, U2 TPS63802DLAR, U4 STM32U585VIT6Q, U5 SE050E2HQ1/Z01Z3Z, U6 TS3USB221ARSER, U7 SN74LVC1G02DBVR(UMW), U8 TPS22917DBVR, U9 TXU0202DCUR

Commit message: Clean DRC: stale copper, sloppy stubs and silk; cleanCopper --check gate
DRC: 0 violations; 3 unconnected (RADIO_TXD, AIRGAP x2) left to the owner.

Copper:
- cleanCopper removed the two "3.3 V vias" connected to nothing: GND stitching
  vias at HEAD, shoved ~2 mm by KiCad's interactive router while the USB pair
  went in; a moved free via takes the net of the plane it lands in. Also four
  pad-less GND tracks (crumbs on stitching vias) and a 0.02 mm USB crumb.
- The owner's stubs: CHG_STAT1's two segments that stopped 0.1 mm short of each
  other joined on their common 45-degree line; two zero-length USB segments and
  a 0.02 mm 0.4 mm-wide BAT sliver lying on its 0.25 mm track removed.
- cleanCopper now drops pad-less GND tracks (a lone GND via is stitching, a GND
  track that reaches no pad is litter) and has --check (exit 1 if anything is
  stale), a gate before every commit.

Silk (14 findings):
- The SE frame drawn around the SE050's first spot ran across its pads: gone
  (two secure elements now; the label names the block).
- Camera-head outline notched clear of mounting hole H1's ring; AIRGAP legend
  0.6 mm up off C_NOR.
- USB-C: wallet:..._BoardEdge, KiCad's land without the outline lines at and
  past the board edge (pads identical, verified); its GCT model entry re-keyed.
- U2's long outline edges are corner marks now (project footprint), clear of
  C_USBSW, whose courtyard leaves no room to move.
syncBoard: --refresh REF re-instantiates an edited library footprint, --board
works on a copy, and a swap keeps the board's text style and each pad's own
settings (the router's solid pour connections). newBoard's legends match.

Gates: nets, AF, sync, pin tables, FPC, lands pass; cleanCopper --check clean;
no GND pad-to-via ties beyond the 9 kept.

Co-Authored-By: Claude Opus 5.5 <noreply@anthropic.com>
Parts:
- J1: footprint Connector_USB:USB_C_Receptacle_HRO_TYPE-C-31-M-12 -> wallet:USB_C_Receptacle_HRO_TYPE-C-31-M-12_BoardEdge
Routing:
- net V3V3: vias 47 -> 45
