File: board/wallet.kicad_pcb (KiCad board)
At the start: 4 copper layers, 48 x 85 mm, 112 parts, among them J1 TYPE-C-31-M-12, U1 BQ25185DLHR, U11 E73-2G4M08S1C, U12 ME6211C28M5G-N, U13 TPS60230RGTR, U14 TLV70313DBVR, U15 MAX17048G+T10, U16 SLS32AIA010MK, U2 TPS63802DLAR, U4 STM32U585VIT6Q, U5 SE050E2HQ1/Z01Z3Z, U6 TS3USB221ARSER, U7 SN74LVC1G02DBVR(UMW), U8 TPS22917DBVR, U9 TXU0202DCUR

Commit message: Board: the flame in ordinary silkscreen on the back, wordmark removed; 3D models applied
- scripts/silkFlame.py prints the Ambire flame across the back in plain
  (single-ink) silkscreen: 45.6 x 68.6 mm, a 0.35 mm gap between facets, cut
  back 0.15 mm from pads, drilled holes and vias, 0.3 mm from the edge and
  slots, 0.5 mm around the human-readable labels (QR CAMERA, SECURE ELEMENT,
  AIRGAP, RADIO, ANT) and 0.15 mm from footprint silkscreen. 67 polygons,
  964 of 1252 mm2 of ink kept. Lives in group FLAME; a rerun replaces it.
- The "AMBIRE" and "Ambire signer · proto 0" texts are removed.
- It runs DRC on a copy (project rules, library table) and installs only if
  the findings do not grow and the board did not change meanwhile: 0/0 before,
  0/0 after. cleanCopper --check: clean.
- art/flame.py: the flame geometry and placement, shared with the concept
  page's preview (pure Python for KiCad's interpreter).
- scripts/applyModels.py --apply: the LCSC models for the power button and the
  camera connector (from board/models.json) are on the footprints now.

Co-Authored-By: Claude Opus 5.5 <noreply@anthropic.com>
Other:
- board text removed: "AMBIRE"
- board text removed: "Ambire signer · proto 0"
