File: board/experiments/radio-gate-west.kicad_pcb (KiCad board)
At the start: 4 copper layers, 48 x 85 mm, 108 parts, among them J1 TYPE-C-31-M-12, U1 BQ25185DLHR, U11 E73-2G4M08S1C, U12 ME6211C28M5G-N, U13 TPS60230RGTR, U14 TLV70313DBVR, U15 MAX17048G+T10, U2 TPS63802DLAR, U4 STM32U585VIT6Q, U5 SE050E2HQ1/Z01Z3Z, U6 TS3USB221ARSER, U7 SN74LVC1G02DBVR(UMW), U8 TPS22917DBVR, U9 TXU0202DCUR

Commit message: TP_NRST next to the MCU's NRST pin
The NRST test pad sat with the other programming pads on the west edge while
NRST is pin 14 on the MCU's east side, behind hand-routed copper: the autorouter
took 29.5 mm down the west edge for it. Now on the front at (33.6, 26.8), beside
NRST's 100 nF cap: 4.7 mm of copper, one via. Same move in the radio-gate
candidate. Unconnected 57 -> 56 on the main board.

Co-Authored-By: Claude Opus 5.5 <noreply@anthropic.com>
Parts:
- moved TP_NRST 29.6 mm to (33.6, 26.8)
Routing:
- net NRST: track 2.34 -> 4.73 mm, vias 0 -> 1
Changed lines of the file:
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@@
 	(footprint "TestPoint:TestPoint_Pad_D1.0mm"
 		(layer "F.Cu")
-		(at 4 25.56)
+		(at 33.6 26.8)
 		(descr "SMD pad as test Point, diameter 1.0mm")
 		(tags "test point SMD pad")
@@
 	)
 	(segment
+		(start 33.6 26.8)
+		(end 33.425 26.8)
+		(width 0.15)
+		(layer "F.Cu")
+		(net "NRST")
+	)
+	(segment
+		(start 33.425 26.8)
+		(end 32.35 27.875)
+		(width 0.15)
+		(layer "F.Cu")
+		(net "NRST")
+	)
+	(via
+		(at 32.35 27.875)
+		(size 0.45)
+		(drill 0.25)
+		(layers "F.Cu" "B.Cu")
+		(net "NRST")
+	)
+	(segment
 		(start 31.89 28.5)
 		(end 31.98 28.41)
@@
 		(width 0.15)
 		(layer "B.Cu")
+		(net "NRST")
+	)
+	(segment
+		(start 32.35 28.04)
+		(end 31.98 28.41)
+		(width 0.15)
+		(layer "B.Cu")
+		(net "NRST")
+	)
+	(segment
+		(start 32.35 27.875)
+		(end 32.35 28.04)
+		(width 0.15)
+		(layer "B.Cu")
